Commit message: Updated MeArm URDF to have joints move correctly. Still no gripper.

File: ros_ws/typeypt/typepyt.urdf (robot description, URDF)
Before this commit: robot typeypt, 6 links, 5 joints
Joints:
- joint elbow: axis 0 1 0 -> 0 -1 0; limit (none) -> lower=0.87 upper=2.44 effort=30 velocity=1.0; origin xyz=0.0 0.0 0.8 rpy=0 0 0 -> xyz=0.0 0.0 0.8 rpy=0 3.36 0; type continuous -> revolute
- joint hip: limit (none) -> lower=0.0 upper=3.14 effort=30 velocity=1.0; origin xyz=0.0 0.0 0.12 rpy=0 0 -1.5707 -> xyz=0.0 0.0 0.12 rpy=0 0 0; type continuous -> revolute
- joint shoulder: limit (none) -> lower=0.52 upper=2.79 effort=30 velocity=1.0; origin xyz=0.2  0.0 0.30 rpy=0 0 0 -> xyz=0.2  0.0 0.30 rpy=0 -1.57 0; type continuous -> revolute
- joint wrist: axis 0 1 0 -> 1 0 0; limit (none) -> lower=0.0 upper=1.57 effort=30 velocity=1.0; type continuous -> revolute
