Commit message: ROS Joint controller outputs but needs an action to set motores.

File: ros_ws/src/typepyt/typepyt.urdf (robot description, URDF)
Before this commit: robot typeypt, 6 links, 5 joints
Joints:
- joint wrist: limit lower=0.0 upper=1.57 effort=30 velocity=1.0 -> lower=0.0 upper=2.7 effort=30 velocity=1.0

Commit message: Pulling in the URDF change from matrhint's fork to see how the system behaves in Gazebo.

File: ros_ws/src/typepyt/typepyt.urdf (robot description, URDF)
Before this commit: robot typeypt, 6 links, 5 joints
Links:
- added link upper_arm2, mass 1.0; collision cylinder length=0.01 radius=0.05; visual cylinder length=0.01 radius=0.05
- link lower_arm: geometry collision cylinder length=0.79 radius=0.05; visual cylinder length=0.79 radius=0.05
Joints:
- added joint elbow1: type revolute, parent upper_arm, child upper_arm2, origin xyz=0.0 0.0 0.8 rpy=0 3.36 0, axis 0 -1 0, limit lower=0.87 upper=2.44 effort=30 velocity=1.0, mimic joint=shoulder multiplier=1 offset=0
- joint elbow: limit lower=0.87 upper=2.44 effort=30 velocity=1.0 -> lower=1.75 upper=3.0 effort=30 velocity=1.0; origin xyz=0.0 0.0 0.8 rpy=0 3.36 0 -> xyz=0.0 0.0 0.01 rpy=0 3.36 0; parent upper_arm -> upper_arm2
